File: Radar1.kicad_sch (KiCad schematic)
At the start: 76 parts, among them J1 USB4215-03-A, J2 Barrel_Jack, U1 BGT24LTR11N16, U10 93LC56B-I/SN, U11 445I23D12M00000, U12 AMM-8211PSM, U2 ADF4159WCCPZ, U3 OPA1656ID, U4 TPS7A2033PDBVR, U5 TPS7A2018PDBVR, U6 TPS7A4700RGWT, U7 FT2232HL-REEL, U8 ADS8353IPW, U9 ADP5600ACPZ-R7, Y1 ECS-TXO-2520MV-500-AN-TR

Commit message: Schematic layout cleanup and resistor value convention
Manual rearrangement/placement pass in KiCad; resistor values switched to
standard k/M convention (e.g. 12kOHMS -> 12k). Netlist verified: 76
components, 58 connected nets unchanged, no annotation errors.

Co-Authored-By: Claude Opus 4.8 <noreply@anthropic.com>
Parts:
- R1: value 12kOHMS -> 12k
- R2: value 10kOHMS -> 10k
Connections:
- net GND: no longer J1.B1/A12 (GND)
Other:
- moved on the sheet: C1, C10, C11, C12, C13, C14, C15, C16, C17, C18, C19, C2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

Commit message: Rev-B fix pass: power/bias corrections from datasheet review
- ADF4159 VP 5V->3.3V (4V abs max), SDVDD tied to +1V8
- U4/U5 6V-max LDOs re-fed from +5V instead of raw VIN
- AMM-8211 Vg moved to ADP5600 regulated -0.505V LDO output;
  Vd1-3 moved to new +3V0_PA net (drain LDO TBD, PGOOD-sequenced)
- FT2232: C1-C3 as VCORE decouplers, VBUS sense divider to RESET#,
  EEPROM DO isolation (R21), MUXOUT pull-up to 3.3V (R22)
- Bulk caps C43-C45, VREF divider stiffened, 29 no-connect flags
- ERC 50 -> 11 errors (rest symbol pin-type quirks + 2 intentional)

Changelog/TODO block on sheet at (318,15).

Co-Authored-By: Claude Fable 5 <noreply@anthropic.com>
Parts:
- added C43, C44: 10uF, symbol Device:C_Small_US
- added C45: 1uF, symbol Device:C_Small_US
- added R20, R22: 10k, symbol Device:R_Small_US
- added R21: 2.2k, symbol Device:R_Small_US
- C16: value 3.3nF -> 3.3uF
- C2: value 10nF -> 100nF
- C3: value 1nF -> 100nF
- R10, R9: value 10k -> 1k
- R17: value 100k -> 0R
- R2: value 10k -> 4.7k
Connections:
- net SDVDD_N is gone; now on net +1V8: C22.1, U2.18 (SDVDD)
- net U9LDO is gone; now on net -VGG: C41.1, U9.7 (LDO_OUT)
- net +1V8: now also C45.1
- net +3V3_RF: now also U2.22 (VP), R22.2; no longer R2.1, U12.14 (Vd3), U12.15 (Vd2), U12.16 (Vd1)
- net +5V: now also U4.1 (IN), U4.3 (EN), U5.1 (IN), U5.3 (EN), C43.1; no longer U2.22 (VP)
- net +VIN: now also C44.1; no longer U4.1 (IN), U4.3 (EN), U5.1 (IN), U5.3 (EN)
- net -VGG: no longer C40.1, U9.11 (CPOUT), U9.8 (CPOUT)
- net ADF_MUXOUT: now also R22.1
- net EE_DATA: now also R21.2; no longer U10.4 (DO)
- net GND: now also C1.2, C2.2, C3.2, J1.B1/A12 (GND), C43.2, C44.2, C45.2, R20.2
- net VCORE: now also C1.1, C2.1, C3.1
- net USB_RESET: now reaches R2.2, U7.14 (~{RESET})
- net USB_RESET: now also R20.1
- net ANT_TX: now reaches U12.10 (RF_OUT)
- net VBUS: now reaches J1.A4/B9 (VBUS)
- net VBUS: now also J1.B4/A9 (VBUS), R2.1
- net ANT_RX: now reaches U1.3 (RX)
- new net +3V0_PA: U12.14 (Vd3), U12.15 (Vd2), U12.16 (Vd1)
- new net EE_DO: R21.1, U10.4 (DO)
- new net VGG_CP: C40.1, U9.11 (CPOUT), U9.8 (CPOUT)
- no-connect marks 19 -> 48
Other:
- note added: "=== REV-B FIXES 2026-07-01 === CHANGED: * ADF4159 VP: 5V -> 3.3V (VP abs max = 4V — was over-stress!) * ADF4159 SDVDD tied to +1V8 (was floating — sigma-delta core unpowered) * U4/U5 (6V-max LDOs) now fed from +5V, not VIN (VIN may exceed 6V) * AMM-8211 Vg now from ADP5600 LDO_OUT = -0.505V, R17=0R (was raw CPOUT = -VIN — would destroy the gate). C40 -> VGG_CP reservoir. * AMM-8211 Vd1-3 moved to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"
- note added: "MUXOUT is 1.8V logic: R22 pulls up to 3.3V — configure MUXOUT open-drain in software. (dig. I/O abs max = AVDD+0.3, so 3.3V OK)"
- note added: "Self-powered USB: RESET# held low until VBUS present via R2 4.7k / R20 10k (FTDI app note AN_146)."
- note added: "TODO: +3V0_PA UNDRIVEN — needs 2.5-3.0V LDO, EN <- U9 PGOOD (gate-before-drain). Do not populate U12 until added."
- note added: "Vg = -0.505V from ADP5600 LDO_OUT (SEL1=SEL2=GND fixed mode, R17=0R). VGG_CP = raw CP out (C40 reservoir). Verify amp Id; trim FB divider if needed."

Commit message: Rev-C: complete functional gaps — PA supply, VREF buffer, rail split
Blockers fixed:
- U13 TPS7A4700 3.0V PA drain LDO drives +3V0_PA (was undriven);
  EN <- U9 PGOOD for gate-before-drain sequencing (AMM-8211 175mA typ)
- U9 ADP5600 re-fed from +5V (5.5V abs max vs raw VIN conflict)
- J3/J4 board-side RF ports for ANT_TX/ANT_RX (2.92mm end-launch;
  stock SMA footprint is a layout placeholder)
- R6 R_TUNE 10k -> 16k per BGT24LTR11 spec for 24.05-24.25GHz VCO

Robustness:
- U16 REF5025 buffered 2.5V -> VREF, replaces R9/R10 divider
  (ADS8353 AINM needs low-Z source; CFR.B7=1 B9=1 pseudo-diff 2xVREF)
- R23/C49 R24/C50 anti-alias RCs (49.9R+10nF) ahead of ADS8353
- U14 TPS7A2033: +3V3_DIG (FT2232/EEPROM) split off +3V3_RF
  (PLL/VCO/TCXO) — was one 300mA LDO near limit with USB noise
- C51 100pF TCXO->REFIN coupling; D1 SS34 reverse-polarity; U15
  TPD2E009 USB ESD; footprints on all passives; sheet A4 -> A3

New symbols in RadarExtra.kicad_sym; full changelog in CHANGELOG.md.
Netlist regression: exact match to expected transform. ERC 11 -> 10
(both intentional Rev-B errors resolved; rest are lib pin-type quirks).

Co-Authored-By: Claude Fable 5 <noreply@anthropic.com>
Parts:
- removed R10, R9: 1k, symbol Device:R_Small_US
- added C46, C47: 10uF, Capacitor_SMD:C_0805_2012Metric, symbol Device:C_Small_US
- added C48, C49, C50: 10nF, Capacitor_SMD:C_0603_1608Metric, symbol Device:C_Small_US
- added C51: 100pF, Capacitor_SMD:C_0603_1608Metric, symbol Device:C_Small_US
- added C52, C53, C54: 1uF, Capacitor_SMD:C_0603_1608Metric, symbol Device:C_Small_US
- added D1: SS34, Diode_SMD:D_SMA, symbol RadarExtra:D_Schottky
- added J3, J4: SMA-2.92mm-EndLaunch, Connector_Coaxial:SMA_Amphenol_132289_EdgeMount, symbol RadarExtra:Conn_Coaxial
- added R23, R24: 49.9R, Resistor_SMD:R_0603_1608Metric, symbol Device:R_Small_US
- added U13: TPS7A4700RGWT, RGW0020A-IPC_A, symbol TPS7A4700RGWT:TPS7A4700RGWT
- added U14: TPS7A2033PDBVR, TPS7A2033PDBVR:SOT95P280X145-5N, symbol TPS7A2033PDBVR:TPS7A2033PDBVR
- added U15: TPD2E009DBZR, Package_TO_SOT_SMD:SOT-23, symbol RadarExtra:TPD2E009
- added U16: REF5025AID, Package_SO:SOIC-8_3.9x4.9mm_P1.27mm, symbol RadarExtra:REF5025
- C1, C10, C11, C12, C13, C14, C15, C17, C18, C19, C2, C20, C21, C22, C23, C24, C26, C28, C29, C3, C30, C31, C32, C33, C34, C35, C36, C37, C38, C39, C4, C41, C42, C45, C5, C6, C7, C8, C9: footprint (none) -> Capacitor_SMD:C_0603_1608Metric
- C16, C25, C27, C40, C43, C44: footprint (none) -> Capacitor_SMD:C_0805_2012Metric
- J2: footprint (none) -> Connector_BarrelJack:BarrelJack_Horizontal
- R1, R11, R12, R13, R14, R15, R16, R17, R18, R19, R2, R20, R21, R22, R3, R4, R5, R7, R8: footprint (none) -> Resistor_SMD:R_0603_1608Metric
- R6: value 10k -> 16k; footprint (none) -> Resistor_SMD:R_0603_1608Metric
Connections:
- net +3V0_PA: now also C47.1, U13.1 (OUT), U13.20 (OUT), U13.3 (SENSE_FB)
- net +3V3_RF: no longer C13.1, C14.1, C15.1, C30.1, C31.1, C32.1, R22.2, U10.8 (VCC), U7.20 (VCCIO-1), U7.31 (VCCIO-2), U7.4 (VPHY), U7.42 (VCCIO-3), U7.50 (VREGIN), U7.56 (VCCIO-4), U7.9 (VPLL)
- net +5V: now also C10.1, U9.1 (VIN), U9.2 (EN), C46.1, C52.1, C54.1, U13.15 (IN), U13.16 (IN), U14.1 (IN), U14.3 (EN), U16.2 (VIN)
- net +VIN: now also D1.2 (K); no longer C10.1, J2.1, U9.1 (VIN), U9.2 (EN)
- net ANT_RX: now also J4.1 (In)
- net ANT_TX: now also J3.1 (In)
- net GND: now also C46.2, C47.2, C48.2, C49.2, C50.2, C52.2, C53.2, C54.2, J3.2 (Ext), J4.2 (Ext), U13.21 (Thermal_Pad), U13.7 (GND), U13.8 (1P6V), U14.2 (GND), U15.3 (GND), U16.4 (GND)
- net IFA_OUT: now also R23.1; no longer U8.1 (AINP_A)
- net IFB_OUT: now also R24.1; no longer U8.8 (AINP_B)
- net REF_CLK: now also C51.1; no longer U2.9 (REFIN)
- net U9PG: now also U13.13 (EN)
- net USB_DM: now also U15.2 (D-)
- net USB_DP: now also U15.1 (D+)
- net VREF: now also U16.6 (VOUT)
- new net +3V3_DIG: C13.1, C14.1, C15.1, C30.1, C31.1, C32.1, C53.1, R22.2, U10.8 (VCC), U14.5 (OUT), U7.20 (VCCIO-1), U7.31 (VCCIO-2), U7.4 (VPHY), U7.42 (VCCIO-3), U7.50 (VREGIN), U7.56 (VCCIO-4), U7.9 (VPLL)
- new net ADC_A: C49.1, R23.2, U8.1 (AINP_A)
- new net ADC_B: C50.1, R24.2, U8.8 (AINP_B)
- new net ADF_REFIN: C51.2, U2.9 (REFIN)
- new net NR_PA: C48.1, U13.14 (NR)
- new net VIN_RAW: D1.1 (A), J2.1
- no-connect marks 48 -> 65
Other:
- note added: "=== REV-C 2026-07-02 (details: CHANGELOG.md) === + U13 3.0V PA drain LDO, EN<-U9 PGOOD (gate-before-drain) + U16 REF5025 buffered 2.5V -> VREF (was R9/R10 divider) + R23/C49 R24/C50 ADC anti-alias (49.9R+10nF, fc~320k) + U14 second 3.3V LDO: +3V3_DIG (FT2232/EEPROM) split from +3V3_RF + C51 100pF TCXO->REFIN; D1 reverse-polarity; U15 USB ESD + J3/J4 RF ports (2.92mm end-launch; SMA footprint = pl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"
- note added: "PA drain rail +3V0_PA: U13 TPS7A4700 set to 3.0V (1P6V ANY-OUT pin grounded: 1.4+1.6V), fed from +5V. EN <- U9 PGOOD (R19 pull-up) so -VGG gate bias is valid before drain power: gate-before-drain sequencing."
- note removed: "TODO: +3V0_PA UNDRIVEN — needs 2.5-3.0V LDO, EN <- U9 PGOOD (gate-before-drain). Do not populate U12 until added."
