File: Radar1.kicad_sch (KiCad schematic)
At the start: 99 parts, among them J1 USB4215-03-A, J2 Barrel_Jack, J3 SMA-2.92mm-EndLaunch, J4 SMA-2.92mm-EndLaunch, U1 BGT24LTR11N16, U10 93LC56B-I/SN, U11 445I23D12M00000, U12 AMM-8211PSM, U13 TPS7A4700RGWT, U14 TPS7A2033PDBVR, U15 TPD2E009DBZR, U16 REF5025AID, U2 ADF4159WCCPZ, U3 OPA1656ID, U4 TPS7A2033PDBVR, U5 TPS7A2018PDBVR, U6 TPS7A4700RGWT, U7 FT2232HL-REEL, U8 ADS8353IPW, U9 ADP5600ACPZ-R7, Y1 ECS-TXO-2520MV-500-AN-TR

Commit message: Footprint pass: RadarFP.pretty with 12 validated vendor footprints, all parts assigned
ERC footprint_link_issues 17->0; netlist connectivity unchanged.

Co-Authored-By: Claude Fable 5 <noreply@anthropic.com>
Parts:
- J1: footprint CONN_8p94X6p5X3p16_12L_GCC -> RadarFP:CONN_8p94X6p5X3p16_12L_GCC
- U1: footprint BGT24LTR11N16:PQFN50P240X240X77-17N-V -> RadarFP:PQFN50P240X240X77-17N-V
- U10: footprint SOIC8-N_MC_MCH -> RadarFP:SOIC8-N_MC_MCH
- U11: footprint 445I23D12M00000_CTS -> RadarFP:445I23D12M00000_CTS
- U13, U6: footprint RGW0020A-IPC_A -> RadarFP:RGW0020A-IPC_A
- U14, U4: footprint TPS7A2033PDBVR:SOT95P280X145-5N -> RadarFP:DBV0005A-IPC_A
- U2: footprint CP_24_10 -> RadarFP:CP_24_10
- U3: footprint D0008A_N -> RadarFP:D0008A_N
- U5: footprint DBV0005A-IPC_A -> RadarFP:DBV0005A-IPC_A
- U7: footprint FT2232HL-REEL:QFP50P1200X1200X160-64N -> RadarFP:QFP50P1200X1200X160-64N
- U8: footprint PW16_TEX -> RadarFP:PW16_TEX
- U9: footprint CP-16-17_ADI -> RadarFP:CP-16-17_ADI
- Y1: footprint ECS-TXO-2520MV-500-AN-TR:OSC_ECS-TXO-2520MV-500-AN-TR -> RadarFP:OSC_ECS-TXO-2520MV-500-AN-TR
Changed lines of the file:
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@@
 			)
 		)
-		(property "Footprint" "PW16_TEX"
+		(property "Footprint" "RadarFP:PW16_TEX"
 			(at 49.53 167.64 0)
 			(effects
@@
 			)
 		)
-		(property "Footprint" "RGW0020A-IPC_A"
+		(property "Footprint" "RadarFP:RGW0020A-IPC_A"
 			(at 340.36 113.03 0)
 			(effects
@@
 			)
 		)
-		(property "Footprint" "ECS-TXO-2520MV-500-AN-TR:OSC_ECS-TXO-2520MV-500-AN-TR"
+		(property "Footprint" "RadarFP:OSC_ECS-TXO-2520MV-500-AN-TR"
 			(at 96.52 92.71 0)
 			(effects
@@
 			)
 		)
-		(property "Footprint" "D0008A_N"
+		(property "Footprint" "RadarFP:D0008A_N"
 			(at 138.43 110.49 0)
 			(effects
@@
 			)
 		)
-		(property "Footprint" "DBV0005A-IPC_A"
+		(property "Footprint" "RadarFP:DBV0005A-IPC_A"
 			(at 20.32 97.79 0)
 			(effects
@@
 			)
 		)
-		(property "Footprint" "FT2232HL-REEL:QFP50P1200X1200X160-64N"
+		(property "Footprint" "RadarFP:QFP50P1200X1200X160-64N"
 			(at 191.77 77.47 0)
 			(effects
@@
 			)
 		)
-		(property "Footprint" "D0008A_N"
+		(property "Footprint" "RadarFP:D0008A_N"
 			(at 270.51 34.29 0)
 			(effects
@@
 			)
 		)
-		(property "Footprint" "CP-16-17_ADI"
+		(property "Footprint" "RadarFP:CP-16-17_ADI"
 			(at 105.41 129.54 0)
 			(effects
@@
 			)
 		)
-		(property "Footprint" "TPS7A2033PDBVR:SOT95P280X145-5N"
+		(property "Footprint" "RadarFP:DBV0005A-IPC_A"
 			(at 340.36 195.58 0)
 			(effects
@@
 			)
 		)
-		(property "Footprint" "RGW0020A-IPC_A"
+		(property "Footprint" "RadarFP:RGW0020A-IPC_A"
 			(at 233.68 118.11 0)
 			(effects
@@
 			)
 		)
-		(property "Footprint" "CONN_8p94X6p5X3p16_12L_GCC"
+		(property "Footprint" "RadarFP:CONN_8p94X6p5X3p16_12L_GCC"
 			(at 51.816 171.196 0)
 			(effects
@@
 			)
 		)
-		(property "Footprint" "TPS7A2033PDBVR:SOT95P280X145-5N"
+		(property "Footprint" "RadarFP:DBV0005A-IPC_A"
 			(at 38.1 76.2 0)
 			(effects
@@
 			)
 		)
-		(property "Footprint" "D0008A_N"
+		(property "Footprint" "RadarFP:D0008A_N"
 			(at 270.51 77.47 0)
 			(effects
@@
 			)
 		)
-		(property "Footprint" "445I23D12M00000_CTS"
+		(property "Footprint" "RadarFP:445I23D12M00000_CTS"
 			(at 173.99 158.75 0)
 			(effects
@@
 			)
 		)
-		(property "Footprint" "SOIC8-N_MC_MCH"
+		(property "Footprint" "RadarFP:SOIC8-N_MC_MCH"
 			(at 22.86 134.62 0)
 			(effects
@@
 			)
 		)
-		(property "Footprint" "CP_24_10"
+		(property "Footprint" "RadarFP:CP_24_10"
 			(at 86.36 24.13 0)
 			(effects
@@
 			)
 		)
-		(property "Footprint" "BGT24LTR11N16:PQFN50P240X240X77-17N-V"
+		(property "Footprint" "RadarFP:PQFN50P240X240X77-17N-V"
 			(at 29.21 19.05 0)
 			(effects
