File: Radar1.kicad_pcb (KiCad board)
At the start: 4 copper layers, 66 x 46 mm, 99 parts, among them J1 USB4215-03-A, J2 Barrel_Jack, J3 SMA-2.92mm-EndLaunch, J4 SMA-2.92mm-EndLaunch, U1 BGT24LTR11N16, U10 93LC56B-I/SN, U11 445I23D12M00000, U12 AMM-8211PSM, U13 TPS7A4700RGWT, U14 TPS7A2033PDBVR, U15 TPD2E009DBZR, U16 REF5025AID, U2 ADF4159WCCPZ, U3 OPA1656ID, U4 TPS7A2033PDBVR, U5 TPS7A2018PDBVR, U6 TPS7A4700RGWT, U7 FT2232HL-REEL, U8 ADS8353IPW, U9 ADP5600ACPZ-R7, Y1 ECS-TXO-2520MV-500-AN-TR

Commit message: Rev-F: IF gain and coupling corner from link budget
Mixer IP1dB (-28 dBm in, 126 mVpk out) mapped onto ADS8353 full scale:
gain x11 -> x19 (R13/R16 = 18k). Coupling C36/C37 100nF -> 560pF: HPF
corner 16 Hz -> 2.8 kHz (min range 1.7 m, kills TX-leakage beat at full
gain). Chain is thermal-noise-limited (190 uV chain vs 44 uV ADC);
detection ~70 m person / ~125 m car per 1 kHz bin at 13 dB; AA corner
limits instrumented range to 191 m. tools/if_link_budget.py reproduces.
Netlist-regression: value-only change, topology untouched.

Co-Authored-By: Claude Fable 5 <noreply@anthropic.com>
Parts:
- C36, C37: value 100nF -> 560pF
- R13, R16: value 10k -> 18k
Changed lines of the file:
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@@
 			)
 		)
-		(property "Value" "10k"
+		(property "Value" "18k"
 			(at 0 1.43 0)
 			(layer "F.Fab")
@@
 			)
 		)
-		(property "Value" "100nF"
+		(property "Value" "560pF"
 			(at 0 1.43 0)
 			(layer "F.Fab")
@@
 			)
 		)
-		(property "Value" "10k"
+		(property "Value" "18k"
 			(at 0 1.43 0)
 			(layer "F.Fab")
@@
 			)
 		)
-		(property "Value" "100nF"
+		(property "Value" "560pF"
 			(at 0 1.43 0)
 			(layer "F.Fab")
